Commit message: getting ready for more complete install instructions

File: urdf/camera.xacro (robot description, xacro)
@@ -6,13 +6,13 @@
   <link name="camera_link">
     <collision>
-            <origin rpy="0 0 0" xyz="0 0 -0.15"/>
+            <origin rpy="0 0 0" xyz="0 0 0"/>
       <geometry>
-    <box size="${camera_link} ${camera_link} ${camera_link}"/>
+    <box size="${camera_link} ${camera_link*2} ${camera_link}"/>
       </geometry>
     </collision>
     <visual>
-            <origin rpy="0 0 0" xyz="0 0 -0.15"/>
+            <origin rpy="0 0 0" xyz="0 0 0"/>
       <geometry>
-    <box size="${camera_link} ${camera_link} ${camera_link}"/>
+    <box size="${camera_link} ${camera_link*2} ${camera_link}"/>
       </geometry>
       <material name="black"/>
@@ -20,5 +20,5 @@
     <inertial>
       <mass value="1e-5" />
-            <origin rpy="0 0 0" xyz="0 0 -0.15"/>
+            <origin rpy="0 0 0" xyz="0 0 0"/>
       <inertia ixx="1e-6" ixy="0" ixz="0" iyy="1e-6" iyz="0" izz="1e-6" />
     </inertial>
@@ -28,5 +28,5 @@
         <parent link="base_link"/>
         <child link="camera_link"/>
-        <origin rpy="0 0 0" xyz="0 0 0.3"/> <!-- moves the child_frame with respect to parent_frame -->
+        <origin rpy="0 0 0" xyz="0.15 0 ${camera_link/2 + 0.15}"/> <!-- moves the child_frame with respect to parent_frame -->
         <limit effort="30" velocity="1.0"/>
     </joint>

File: urdf/main.xacro (robot description, xacro)
@@ -1,4 +1,16 @@
 <?xml version="1.0"?>
 <robot xmlns:xacro="http://www.ros.org/wiki/xacro" name="growbot">
+    <xacro:include filename="$(find growbot_simulations)/urdf/wheel.xacro" />
+    <xacro:include filename="$(find growbot_simulations)/urdf/camera.xacro" />
+    <xacro:include filename="$(find growbot_simulations)/urdf/plugins.xacro" />
+  <material name="silver">
+    <color rgba="0.5 0.5 0.5 1"/>
+  </material>
+  <material name="black">
+    <color rgba="0 0 0 1"/>
+  </material>
+  <material name="yellow">
+    <color rgba="1 1 0 1"/>
+  </material>
   <xacro:property name="body_len" value="0.4" />
   <xacro:property name="body_width" value="0.4" />
@@ -10,16 +22,4 @@
   <xacro:property name="wheel_z_offset" value="-0.17" />
   <xacro:property name="mass" value="7" />
-  <material name="silver">
-    <color rgba="0.5 0.5 0.5 1"/>
-  </material>
-    <material name="black">
-    <color rgba="0 0 0 1"/>
-  </material>
-    <material name="yellow">
-    <color rgba="1 1 0 1"/>
-  </material>
-    <xacro:include filename="$(find growbot_simulations)/urdf/wheel.xacro" />
-    <xacro:include filename="$(find growbot_simulations)/urdf/camera.xacro" />
-    <xacro:include filename="$(find growbot_simulations)/urdf/plugins.xacro" />
   <!-- dummy link and joint added to fix inertial error per [https://answers.ros.org/question/192817/error-msg-the-root-link_base-has-an-inertia-specified-in-the-urdf-but-kdl/] -->
   <link name="dummy">
@@ -59,4 +59,5 @@
   <xacro:wheel prefix="back_right" x_offset="${-wheel_x_offset}" y_offset="${wheel_y_offset}" z_offset="${wheel_z_offset}" width="${wheel_width}" radius="${wheel_diam/2}" y_reflect="-1" />
   <xacro:wheel prefix="back_left"  x_offset="${-wheel_x_offset}" y_offset="${wheel_y_offset}" z_offset="${wheel_z_offset}" width="${wheel_width}" radius="${wheel_diam/2}" y_reflect="1" />
-<xacro:camera />
+      <!-- TODO: send variables to camera script to allow for parametric camera size/location -->
+  <xacro:camera />
 </robot>

Commit message: camera works, but movement program is broke

File: urdf/camera.xacro (robot description, xacro)
@@ -2,5 +2,5 @@
 <robot xmlns:xacro="http://www.ros.org/wiki/xacro" name="my_robot">
 <xacro:macro name="camera">
-    <xacro:property name="camera_link" value="0.05" /> <!-- Size of square 'camera' box -->
+    <xacro:property name="camera_size" value="0.05" /> <!-- Size of square 'camera' box -->
     <!-- Camera -->
   <link name="camera_link">
@@ -8,5 +8,5 @@
             <origin rpy="0 0 0" xyz="0 0 0"/>
       <geometry>
-    <box size="${camera_link} ${camera_link*2} ${camera_link}"/>
+    <box size="${camera_size} ${camera_size*2} ${camera_size}"/>
       </geometry>
     </collision>
@@ -14,5 +14,5 @@
             <origin rpy="0 0 0" xyz="0 0 0"/>
       <geometry>
-    <box size="${camera_link} ${camera_link*2} ${camera_link}"/>
+    <box size="${camera_size} ${camera_size*2} ${camera_size}"/>
       </geometry>
       <material name="black"/>
@@ -23,10 +23,21 @@
       <inertia ixx="1e-6" ixy="0" ixz="0" iyy="1e-6" iyz="0" izz="1e-6" />
     </inertial>
+</link>
+  <!-- generate an optical frame http://www.ros.org/reps/rep-0103.html#suffix-frames
+      so that ros and opencv can operate on the camera frame correctly -->
+  <joint name="camera_optical_joint" type="fixed">
+    <!-- these values have to be these values otherwise the gazebo camera image
+        won't be aligned properly with the frame it is supposedly originating from -->
+    <origin xyz="0 0 0" rpy="${-pi/2} 0 ${-pi/2}"/>
+    <parent link="camera_link"/>
+    <child link="camera_link_optical"/>
+  </joint>
+  <link name="camera_link_optical">
   </link>
-    <joint name="base_to_camera" type="continuous">
+    <joint name="chassis_to_camera" type="fixed">
         <axis xyz="0 0 1"/>  <!-- changes axis of rotation -->
-        <parent link="base_link"/>
+        <parent link="chassis_link"/>
         <child link="camera_link"/>
-        <origin rpy="0 0 0" xyz="0.15 0 ${camera_link/2 + 0.15}"/> <!-- moves the child_frame with respect to parent_frame -->
+        <origin rpy="0 0 0" xyz="0.15 0 ${camera_size/2 + 0.15}"/> <!-- moves the child_frame with respect to parent_frame -->
         <limit effort="30" velocity="1.0"/>
     </joint>
@@ -36,48 +47,8 @@
             <mechanicalReduction>1</mechanicalReduction>
         </actuator>
-        <joint name="base_to_camera">
+        <joint name="chassis_to_camera">
             <hardwareInterface>hardware_interface/PositionJointInterface</hardwareInterface>
         </joint>
     </transmission>
 </xacro:macro>
-  <!--Gazebo Camera Plugin-->
-   <gazebo reference="camera">
-    <sensor type="camera" name="camera">
-      <update_rate>30.0</update_rate>
-      <camera name="head">
-        <horizontal_fov>1.3962634</horizontal_fov>
-        <image>
-          <width>800</width>
-          <height>800</height>
-          <format>R8G8B8</format>
-        </image>
-        <clip>
-          <near>0.02</near>
-          <far>300</far>
-        </clip>
-        <noise>
-          <type>gaussian</type>
-          <!-- Noise is sampled independently per pixel on each frame.
-               That pixel's noise value is added to each of its color
-               channels, which at that point lie in the range [0,1]. -->
-          <mean>0.0</mean>
-          <stddev>0.007</stddev>
-        </noise>
-      </camera>
-      <plugin name="camera_controller" filename="libgazebo_ros_camera.so">
-        <alwaysOn>true</alwaysOn>
-        <updateRate>0.0</updateRate>
-        <cameraName>/growbot/camera</cameraName>
-        <imageTopicName>image_raw</imageTopicName>
-        <cameraInfoTopicName>camera_info</cameraInfoTopicName>
-        <frameName>camera</frameName>
-        <hackBaseline>0.07</hackBaseline>
-        <distortionK1>0.0</distortionK1>
-        <distortionK2>0.0</distortionK2>
-        <distortionK3>0.0</distortionK3>
-        <distortionT1>0.0</distortionT1>
-        <distortionT2>0.0</distortionT2>
-      </plugin>
-    </sensor>
-  </gazebo>
-</robot>
+ </robot>

File: urdf/main.xacro (robot description, xacro)
@@ -3,5 +3,6 @@
     <xacro:include filename="$(find growbot_simulations)/urdf/wheel.xacro" />
     <xacro:include filename="$(find growbot_simulations)/urdf/camera.xacro" />
-    <xacro:include filename="$(find growbot_simulations)/urdf/plugins.xacro" />
+    <!--<xacro:include filename="$(find growbot_simulations)/urdf/plugins.xacro" />-->
+    <xacro:include filename="$(find growbot_simulations)/urdf/growbot.gazebo" />
   <material name="silver">
     <color rgba="0.5 0.5 0.5 1"/>
@@ -23,7 +24,7 @@
   <xacro:property name="mass" value="7" />
   <!-- dummy link and joint added to fix inertial error per [https://answers.ros.org/question/192817/error-msg-the-root-link_base-has-an-inertia-specified-in-the-urdf-but-kdl/] -->
-  <link name="dummy">
+  <link name="dummy_link">
   </link>
-    <link name="base_link">
+    <link name="chassis_link">
         <visual>
             <geometry>
@@ -52,6 +53,6 @@
       <!-- dummy link and joint added to fix inertial error per [https://answers.ros.org/question/192817/error-msg-the-root-link_base-has-an-inertia-specified-in-the-urdf-but-kdl/] -->
   <joint name="dummy_joint" type="fixed">
-     <parent link="dummy"/>
-     <child link="base_link"/>
+     <parent link="dummy_link"/>
+     <child link="chassis_link"/>
   </joint>
   <xacro:wheel prefix="front_right" x_offset="${wheel_x_offset}" y_offset="${wheel_y_offset}" z_offset="${wheel_z_offset}" width="${wheel_width}" radius="${wheel_diam/2}" y_reflect="-1" />

File: urdf/plugins.xacro (robot description, xacro)
@@ -1,4 +1,4 @@
 <?xml version="1.0"?>
-<robot>
+<robot name="growbot" xmlns:xacro="http://ros.org/wiki/xacro">
     <!-- Add ROS plugin so we can interact with our robot -->
     <gazebo>
@@ -37,5 +37,5 @@
         <imageTopicName>image_raw</imageTopicName>
         <cameraInfoTopicName>camera_info</cameraInfoTopicName>
-        <frameName>camera</frameName>
+        <frameName>camera_link_optical</frameName>
         <hackBaseline>0.07</hackBaseline>
         <distortionK1>0.0</distortionK1>

File: urdf/wheel.xacro (robot description, xacro)
@@ -25,7 +25,7 @@
         </inertial>
     </link>
-    <joint name="base_to_${prefix}_wheel" type="continuous">
+    <joint name="chassis_to_${prefix}_wheel" type="continuous">
         <axis xyz="0 1 0"/>
-        <parent link="base_link"/>
+        <parent link="chassis_link"/>
         <child link="${prefix}_wheel"/>
         <origin rpy="0 0 0" xyz="${x_offset} ${y_reflect*y_offset} ${z_offset}"/> <!-- move the child_frame with respect to parent_frame -->
@@ -37,5 +37,5 @@
             <mechanicalReduction>1</mechanicalReduction>
         </actuator>
-        <joint name="base_to_${prefix}_wheel">
+        <joint name="chassis_to_${prefix}_wheel">
             <hardwareInterface>hardware_interface/VelocityJointInterface</hardwareInterface>
         </joint>

Commit message: driving no work

File: urdf/camera.xacro (robot description, xacro)
@@ -1,4 +1,4 @@
 <?xml version="1.0"?>
-<robot xmlns:xacro="http://www.ros.org/wiki/xacro" name="my_robot">
+<robot xmlns:xacro="http://www.ros.org/wiki/xacro" name="growbot">
 <xacro:macro name="camera">
     <xacro:property name="camera_size" value="0.05" /> <!-- Size of square 'camera' box -->
@@ -39,5 +39,5 @@
         <parent link="chassis_link"/>
         <child link="camera_link"/>
-        <origin rpy="0 0 0" xyz="0.15 0 ${camera_size/2 + 0.15}"/> <!-- moves the child_frame with respect to parent_frame -->
+        <origin rpy="0 0 0" xyz="${camera_size/2 + 0.15} 0 ${camera_size/2 + 0.15}"/> <!-- moves the child_frame with respect to parent_frame -->
         <limit effort="30" velocity="1.0"/>
     </joint>

File: urdf/main.xacro (robot description, xacro)
@@ -62,3 +62,9 @@
       <!-- TODO: send variables to camera script to allow for parametric camera size/location -->
   <xacro:camera />
+    <!-- Add ROS plugin so we can interact with our robot -->
+  <gazebo>
+      <plugin name="gazebo_ros_control" filename="libgazebo_ros_control.so">
+          <!--<robotNamespace>/growbot</robotNamespace>-->
+      </plugin>
+  </gazebo>
 </robot>

Commit message: working!

File: urdf/camera.xacro (robot description, xacro)
@@ -1,4 +1,4 @@
 <?xml version="1.0"?>
-<robot xmlns:xacro="http://www.ros.org/wiki/xacro" name="my_robot">
+<robot xmlns:xacro="http://www.ros.org/wiki/xacro" name="growbot">
 <xacro:macro name="camera">
     <xacro:property name="camera_link" value="0.05" /> <!-- Size of square 'camera' box -->
@@ -24,4 +24,15 @@
     </inertial>
   </link>
+  <!-- generate an optical frame http://www.ros.org/reps/rep-0103.html#suffix-frames
+      so that ros and opencv can operate on the camera frame correctly -->
+  <joint name="camera_optical_joint" type="fixed">
+    <!-- these values have to be these values otherwise the gazebo camera image
+        won't be aligned properly with the frame it is supposedly originating from -->
+    <origin xyz="0 0 0" rpy="${-pi/2} 0 ${-pi/2}"/>
+    <parent link="camera_link"/>
+    <child link="camera_link_optical"/>
+  </joint>
+  <link name="camera_link_optical">
+   </link>
     <joint name="base_to_camera" type="continuous">
         <axis xyz="0 0 1"/>  <!-- changes axis of rotation -->

File: urdf/main.xacro (robot description, xacro)
@@ -4,4 +4,5 @@
     <xacro:include filename="$(find growbot_simulations)/urdf/camera.xacro" />
     <xacro:include filename="$(find growbot_simulations)/urdf/plugins.xacro" />
+    <xacro:include filename="$(find growbot_simulations)/urdf/growbot.gazebo" />
   <material name="silver">
     <color rgba="0.5 0.5 0.5 1"/>

File: urdf/plugins.xacro (robot description, xacro)
@@ -9,5 +9,5 @@
   <!--Gazebo Camera Plugin-->
    <gazebo reference="camera">
-    <sensor type="camera" name="camera">
+    <sensor type="camera" name="camera2">
       <update_rate>30.0</update_rate>
       <camera name="head">
@@ -34,5 +34,5 @@
         <alwaysOn>true</alwaysOn>
         <updateRate>0.0</updateRate>
-        <cameraName>/growbot/camera</cameraName>
+        <cameraName>/growbot/camera2</cameraName>
         <imageTopicName>image_raw</imageTopicName>
         <cameraInfoTopicName>camera_info</cameraInfoTopicName>

Commit message: Idk, but rviz no work now

File: urdf/camera.xacro (robot description, xacro)
@@ -35,7 +35,7 @@
   <link name="camera_link_optical">
    </link>
-    <joint name="base_to_camera" type="continuous">
+    <joint name="chassis_to_camera" type="continuous">
         <axis xyz="0 0 1"/>  <!-- changes axis of rotation -->
-        <parent link="base_link"/>
+        <parent link="chassis_link"/>
         <child link="camera_link"/>
         <origin rpy="0 0 0" xyz="0.15 0 ${camera_link/2 + 0.15}"/> <!-- moves the child_frame with respect to parent_frame -->
@@ -47,5 +47,5 @@
             <mechanicalReduction>1</mechanicalReduction>
         </actuator>
-        <joint name="base_to_camera">
+        <joint name="chassis_to_camera">
             <hardwareInterface>hardware_interface/PositionJointInterface</hardwareInterface>
         </joint>

File: urdf/main.xacro (robot description, xacro)
@@ -24,7 +24,7 @@
   <xacro:property name="mass" value="7" />
   <!-- dummy link and joint added to fix inertial error per [https://answers.ros.org/question/192817/error-msg-the-root-link_base-has-an-inertia-specified-in-the-urdf-but-kdl/] -->
-  <link name="dummy">
+  <link name="dummy_link">
   </link>
-    <link name="base_link">
+    <link name="chassis_link">
         <visual>
             <geometry>
@@ -53,6 +53,6 @@
       <!-- dummy link and joint added to fix inertial error per [https://answers.ros.org/question/192817/error-msg-the-root-link_base-has-an-inertia-specified-in-the-urdf-but-kdl/] -->
   <joint name="dummy_joint" type="fixed">
-     <parent link="dummy"/>
-     <child link="base_link"/>
+     <parent link="dummy_link"/>
+     <child link="chassis_link"/>
   </joint>
   <xacro:wheel prefix="front_right" x_offset="${wheel_x_offset}" y_offset="${wheel_y_offset}" z_offset="${wheel_z_offset}" width="${wheel_width}" radius="${wheel_diam/2}" y_reflect="-1" />
